Commit message: Fixed atlas URDF

File: robots/atlas/urdf/atlas.urdf (robot description, URDF)
Before this commit: robot drc_skeleton, 44 links, 43 joints
Links:
- link head: geometry visual mesh filename=../meshes/head.stl
- link l_clav: geometry collision box size=0.1 0.07 0.072; visual mesh filename=../meshes/r_clav.stl
- link l_foot: geometry collision box size=0.1 0.08 0.02; collision box size=0.227 0.133887 0.05
- link l_larm: geometry collision box size=0.025 0.06 0.06; collision box size=0.025 0.155 0.07
- link l_lfarm: geometry collision cylinder length=0.015 radius=0.045; collision cylinder length=0.015 radius=0.052
- link l_lglut: geometry visual mesh filename=../meshes/l_lglut.stl
- link l_lleg: geometry collision cylinder length=0.40 radius=0.07; visual mesh filename=../meshes/l_lleg.stl
- link l_scap: geometry collision box size=0.02 0.029 0.018; collision box size=0.028 0.090 0.05
- link l_talus: geometry collision cylinder length=0.010059 radius=0.010348; collision cylinder length=0.029542 radius=0.010181
- link l_uarm: geometry collision box size=0.05 0.07 0.15; collision cylinder length=0.11 radius=0.065
- link l_ufarm: geometry collision box size=0.08 0.09 0.11; collision cylinder length=0.1 radius=0.053
- link l_uglut: geometry visual mesh filename=../meshes/l_uglut.stl
- link l_uleg: geometry collision box size=0.07 0.038 0.14; collision box size=0.07 0.038 0.15
- link ltorso: geometry visual mesh filename=../meshes/ltorso.stl
- link mtorso: geometry visual mesh filename=../meshes/mtorso.stl
- link pelvis: geometry collision cylinder length=0.05 radius=0.16; collision cylinder length=0.05 radius=0.16
- link r_clav: geometry collision box size=0.1 0.07 0.072; collision cylinder length=0.1525 radius=0.0555
- link r_foot: geometry collision box size=0.1 0.08 0.02; collision box size=0.227 0.133887 0.05
- link r_larm: geometry collision box size=0.025 0.06 0.06; collision box size=0.025 0.155 0.07
- link r_lfarm: geometry collision cylinder length=0.015 radius=0.045; collision cylinder length=0.015 radius=0.052
- link r_lglut: geometry visual mesh filename=../meshes/r_lglut.stl
- link r_lleg: geometry collision cylinder length=0.40 radius=0.07; visual mesh filename=../meshes/r_lleg.stl
- link r_scap: geometry collision box size=0.02 0.029 0.018; collision box size=0.028 0.090 0.05
- link r_talus: geometry collision cylinder length=0.010059 radius=0.010348; collision cylinder length=0.029542 radius=0.010181
- link r_uarm: geometry collision box size=0.05 0.07 0.15; collision cylinder length=0.11 radius=0.065
- link r_ufarm: geometry collision cylinder length=0.1 radius=0.053; collision cylinder length=0.125 radius=0.040
- link r_uglut: geometry visual mesh filename=../meshes/r_uglut.stl
- link r_uleg: geometry collision box size=0.07 0.038 0.14; collision box size=0.07 0.038 0.15
- link utorso: geometry collision box size=0.13 0.50 0.10; collision box size=0.2 0.18 0.10

Commit message: Working on Atlas stuff and fixing the solo12 cyclic demo

File: robots/atlas/urdf/atlas.urdf (robot description, URDF)
Before this commit: robot drc_skeleton, 44 links, 43 joints
Links:
- added link l_foot_ee0, mass 0.0; visual sphere radius=0.015
- added link l_foot_ee1, mass 0.0; visual sphere radius=0.015
- added link l_foot_ee2, mass 0.0; visual sphere radius=0.015
- added link l_foot_ee3, mass 0.0; visual sphere radius=0.015
- added link r_foot_ee0, mass 0.0; visual sphere radius=0.015
- added link r_foot_ee1, mass 0.0; visual sphere radius=0.015
- added link r_foot_ee2, mass 0.0; visual sphere radius=0.015
- added link r_foot_ee3, mass 0.0; visual sphere radius=0.015
Joints:
- added joint l_leg_ee0: type fixed, parent l_talus, child l_foot_ee0, origin xyz=0.17 -0.03 -0.08 rpy=0 0 0
- added joint l_leg_ee1: type fixed, parent l_talus, child l_foot_ee1, origin xyz=0.17 0.03 -0.08 rpy=0 0 0
- added joint l_leg_ee2: type fixed, parent l_talus, child l_foot_ee2, origin xyz=-0.09 -0.035 -0.08 rpy=0 0 0
- added joint l_leg_ee3: type fixed, parent l_talus, child l_foot_ee3, origin xyz=-0.09 0.035 -0.08 rpy=0 0 0
- added joint r_leg_ee0: type fixed, parent r_talus, child r_foot_ee0, origin xyz=0.17 -0.03 -0.08 rpy=0 0 0
- added joint r_leg_ee1: type fixed, parent r_talus, child r_foot_ee1, origin xyz=0.17 0.03 -0.08 rpy=0 0 0
- added joint r_leg_ee2: type fixed, parent r_talus, child r_foot_ee2, origin xyz=-0.09 -0.035 -0.08 rpy=0 0 0
- added joint r_leg_ee3: type fixed, parent r_talus, child r_foot_ee3, origin xyz=-0.09 0.035 -0.08 rpy=0 0 0
